File: 68000_afterWireing.sch (EAGLE design)
At the start: 19 parts, among them IC1 74LS32N, IC2 74LS04N, IC3 74LS04N, X1 22-23-2021

Commit message: Fixed errors and warnings after first autoroute. But Need to move components because their are still airwires after autorouting
Parts:
- removed CLK_OSCILLATOR: ASE, crystal:ASE
- added QG1: SG-615PTW, crystal:SG-615PTW
Connections:
- net GND: now also 6821_IOP.VSS, QG1.GND; no longer CLK_OSCILLATOR.GND
- net N$10: now also MC68000G$1.DTACK
- net N$16: now also D1.A
- net N$26: now also QG1.FO
- net N$6: now also 6821_IOA.E
- net VCC: now also 6821_IOP.VCC, QG1.VCC; no longer CLK_OSCILLATOR.VDD
Other:
- moved on the sheet: D1, RESET_SWITCH

Commit message: FINAL: Sent to Bay Area Circuits
Parts:
- removed QG1: SG-615PTW, crystal:SG-615PTW
- added U$1: TTL_OSCILLATOR, TTL_OSCILLATOR:TTL_OSCILLATOR
- renumbered 2732EVEN_EPROM to 2732_ODD, 2732ODD_EPROM to 2732_EVEN, 6821_IO to 6821_ODD
Connections:
- net GND: now also U$1.P$7; no longer QG1.GND
- net N$26: now also U$1.P$8; no longer QG1.FO
- net VCC: now also MC68000G$1.BERR, MC68000G$1.BGACK, MC68000G$1.BR, MC68000G$1.IPL0, MC68000G$1.IPL1, MC68000G$1.IPL2, U$1.P$14; no longer QG1.VCC
Other:
- note added: "MC68000 A0-D7"
- note added: "MC68000 A1-A12"
- note added: "MC68000 D0-D7"
- note added: "MC68000 D8-D15"
